File: megarom.kicad_sch (KiCad schematic)
At the start: 17 parts, among them P1 CONN_MSXSLOT_ALIGNED, P2 CONN_02X07, P7 CONN_02X07, P8 CONN_01X02, U1 74LS32, U2 74LS670, U3 74LS670, U4 39SF040, U5 74LS157, U6 74LS157

Commit message: Added title, data, revision and comments to the schematics
Other:
- title: (none) -> MSX megarom cartridge with TTL components
Changed lines of the file:
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@@
 (kicad_sch (version 20211123) (generator eeschema)
   (paper "A4")
+  (title_block
+    (title "MSX megarom cartridge with TTL components")
+    (date "2022-04-21")
+    (rev "0.1")
+    (comment 1 "Designed by Sangwoo Shim")
+    (comment 2 "https://github.com/borishim/msx-megarom")
+  )
   (junction (at 35.56 139.7) (diameter 0) (color 0 0 0 0)
   )
